File: src/HInata-debug-board.sch (EAGLE design)
At the start: 0 parts

Commit message: fix Hinata-debug-board
Parts:
- added D_LEFT, D_RIGHT: (no value), pinhead:PINHD-1X4
- added MCU_LEFT, MCU_RIGHT: (no value), pinhead:PINHD-1X15
- added U_LEFT, U_RIGHT: (no value), pinhead:PINHD-1X2
Connections:
- new net 5V: D_LEFT.4, MCU_RIGHT.4
- new net COM_LED: D_LEFT.3, MCU_RIGHT.11
- new net CS: D_RIGHT.1, MCU_RIGHT.9
- new net GND: D_LEFT.1, MCU_RIGHT.2, U_LEFT.1, U_LEFT.2, U_RIGHT.1, U_RIGHT.2
- new net INT: D_LEFT.2, MCU_RIGHT.10
- new net MISO: D_RIGHT.2, MCU_RIGHT.7
- new net MOSI: D_RIGHT.3, MCU_RIGHT.6
- new net SCK: D_RIGHT.4, MCU_RIGHT.15
Other:
- note added: "MCU_F303K8"
- note added: "ひなた"
Changed lines of the file:
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@@
 <parts>
 <part name="FRAME1" library="frames" library_urn="urn:adsk.eagle:library:229" deviceset="A3L-LOC" device=""/>
+<part name="MCU_LEFT" library="pinhead" library_urn="urn:adsk.eagle:library:325" deviceset="PINHD-1X15" device="" package3d_urn="urn:adsk.eagle:package:22424/2"/>
+<part name="MCU_RIGHT" library="pinhead" library_urn="urn:adsk.eagle:library:325" deviceset="PINHD-1X15" device="" package3d_urn="urn:adsk.eagle:package:22424/2"/>
+<part name="P+1" library="supply1" library_urn="urn:adsk.eagle:library:371" deviceset="VCC" device=""/>
+<part name="SUPPLY1" library="supply2" library_urn="urn:adsk.eagle:library:372" deviceset="GND" device=""/>
+<part name="D_LEFT" library="pinhead" library_urn="urn:adsk.eagle:library:325" deviceset="PINHD-1X4" device="" package3d_urn="urn:adsk.eagle:package:22407/2"/>
+<part name="D_RIGHT" library="pinhead" library_urn="urn:adsk.eagle:library:325" deviceset="PINHD-1X4" device="" package3d_urn="urn:adsk.eagle:package:22407/2"/>
+<part name="U_LEFT" library="pinhead" library_urn="urn:adsk.eagle:library:325" deviceset="PINHD-1X2" device="" package3d_urn="urn:adsk.eagle:package:22435/2"/>
+<part name="U_RIGHT" library="pinhead" library_urn="urn:adsk.eagle:library:325" deviceset="PINHD-1X2" device="" package3d_urn="urn:adsk.eagle:package:22435/2"/>
+<part name="P+2" library="supply1" library_urn="urn:adsk.eagle:library:371" deviceset="VCC" device=""/>
+<part name="SUPPLY2" library="supply2" library_urn="urn:adsk.eagle:library:372" deviceset="GND" device=""/>
 </parts>
 <sheets>
 <sheet>
 <plain>
+<wire x1="147.32" y1="162.56" x2="147.32" y2="101.6" width="0.1524" layer="97"/>
+<wire x1="147.32" y1="101.6" x2="210.82" y2="101.6" width="0.1524" layer="97"/>
+<wire x1="210.82" y1="101.6" x2="210.82" y2="162.56" width="0.1524" layer="97"/>
+<wire x1="210.82" y1="162.56" x2="147.32" y2="162.56" width="0.1524" layer="97"/>
+<text x="149.86" y="154.94" size="3.81" layer="97">MCU_F303K8</text>
+<wire x1="218.44" y1="162.56" x2="218.44" y2="101.6" width="0.1524" layer="97"/>
+<wire x1="218.44" y1="101.6" x2="279.4" y2="101.6" width="0.1524" layer="97"/>
+<wire x1="279.4" y1="101.6" x2="279.4" y2="162.56" width="0.1524" layer="97"/>
+<wire x1="279.4" y1="162.56" x2="218.44" y2="162.56" width="0.1524" layer="97"/>
+<text x="223.52" y="154.94" size="3.81" layer="97">ひなた</text>
 </plain>
 <instances>
@@
 <attribute name="SHEET" x="357.505" y="5.08" size="2.54" layer="94"/>
 </instance>
+<instance part="MCU_LEFT" gate="A" x="177.8" y="127" smashed="yes">
+<attribute name="NAME" x="163.83" y="147.955" size="1.778" layer="95"/>
+<attribute name="VALUE" x="171.45" y="104.14" size="1.778" layer="96"/>
+</instance>
+<instance part="MCU_RIGHT" gate="A" x="180.34" y="127" smashed="yes" rot="MR0">
+<attribute name="NAME" x="196.85" y="147.955" size="1.778" layer="95" rot="MR0"/>
+<attribute name="VALUE" x="186.69" y="104.14" size="1.778" layer="96" rot="MR0"/>
+</instance>
+<instance part="P+1" gate="VCC" x="198.12" y="142.24" smashed="yes"/>
+<instance part="SUPPLY1" gate="GND" x="190.5" y="139.7" smashed="yes">
+<attribute name="VALUE" x="187.833" y="137.541" size="1.778" layer="96"/>
+</instance>
+<instance part="D_LEFT" gate="A" x="248.92" y="124.46" smashed="yes">
+<attribute name="NAME" x="240.03" y="132.715" size="1.778" layer="95"/>
+<attribute name="VALUE" x="242.57" y="116.84" size="1.778" layer="96"/>
+</instance>
+<instance part="D_RIGHT" gate="A" x="251.46" y="124.46" smashed="yes" rot="MR0">
+<attribute name="NAME" x="262.89" y="132.715" size="1.778" layer="95" rot="MR0"/>
+<attribute name="VALUE" x="257.81" y="116.84" size="1.778" layer="96" rot="MR0"/>
+</instance>
+<instance part="U_LEFT" gate="G$1" x="248.92" y="134.62" smashed="yes">
+<attribute name="NAME" x="240.03" y="140.335" size="1.778" layer="95"/>
+<attribute name="VALUE" x="242.57" y="129.54" size="1.778" layer="96"/>
+</instance>
+<instance part="U_RIGHT" gate="G$1" x="251.46" y="134.62" smashed="yes" rot="MR0">
+<attribute name="NAME" x="262.89" y="140.335" size="1.778" layer="95" rot="MR0"/>
+<attribute name="VALUE" x="257.81" y="129.54" size="1.778" layer="96" rot="MR0"/>
+</instance>
+<instance part="P+2" gate="VCC" x="231.14" y="124.46" smashed="yes"/>
+<instance part="SUPPLY2" gate="GND" x="228.6" y="111.76" smashed="yes">
+<attribute name="VALUE" x="225.933" y="109.601" size="1.778" layer="96"/>
+</instance>
 </instances>
 <busses>
 </busses>
 <nets>
+<net name="MOSI" class="0">
+<segment>
+<pinref part="MCU_RIGHT" gate="A" pin="6"/>
+<wire x1="182.88" y1="132.08" x2="195.58" y2="132.08" width="0.1524" layer="91"/>
+<label x="187.96" y="132.08" size="1.778" layer="95"/>
+</segment>
+<segment>
+<pinref part="D_RIGHT" gate="A" pin="3"/>
+<wire x1="254" y1="124.46" x2="266.7" y2="124.46" width="0.1524" layer="91"/>
+<label x="259.08" y="124.46" size="1.778" layer="95"/>
+</segment>
+</net>
+<net name="MISO" class="0">
+<segment>
+<pinref part="MCU_RIGHT" gate="A" pin="7"/>
+<wire x1="182.88" y1="129.54" x2="195.58" y2="129.54" width="0.1524" layer="91"/>
+<label x="187.96" y="129.54" size="1.778" layer="95"/>
+</segment>
+<segment>
+<pinref part="D_RIGHT" gate="A" pin="2"/>
+<wire x1="254" y1="127" x2="266.7" y2="127" width="0.1524" layer="91"/>
+<label x="259.08" y="127" size="1.778" layer="95"/>
+</segment>
+</net>
+<net name="SCK" class="0">
+<segment>
+<pinref part="D_RIGHT" gate="A" pin="4"/>
+<wire x1="254" y1="121.92" x2="266.7" y2="121.92" width="0.1524" layer="91"/>
+<label x="259.08" y="121.92" size="1.778" layer="95"/>
+</segment>
+<segment>
+<pinref part="MCU_RIGHT" gate="A" pin="15"/>
+<wire x1="182.88" y1="109.22" x2="195.58" y2="109.22" width="0.1524" layer="91"/>
+<label x="187.96" y="109.22" size="1.778" layer="95"/>
+</segment>
+</net>
+<net name="CS" class="0">
+<segment>
+<pinref part="MCU_RIGHT" gate="A" pin="9"/>
+<wire x1="182.88" y1="124.46" x2="195.58" y2="124.46" width="0.1524" layer="91"/>
+<label x="190.5" y="124.46" size="1.778" layer="95"/>
+</segment>
+<segment>
+<pinref part="D_RIGHT" gate="A" pin="1"/>
+<wire x1="254" y1="129.54" x2="266.7" y2="129.54" width="0.1524" layer="91"/>
+<label x="259.08" y="129.54" size="1.778" layer="95"/>
+</segment>
+</net>
+<net name="INT" class="0">
+<segment>
+<pinref part="MCU_RIGHT" gate="A" pin="10"/>
+<wire x1="182.88" y1="121.92" x2="195.58" y2="121.92" width="0.1524" layer="91"/>
+<label x="190.5" y="121.92" size="1.778" layer="95"/>
+</segment>
+<segment>
+<pinref part="D_LEFT" gate="A" pin="2"/>
+<wire x1="246.38" y1="127" x2="233.68" y2="127" width="0.1524" layer="91"/>
+<label x="236.22" y="127" size="1.778" layer="95"/>
+</segment>
+</net>
+<net name="COM_LED" class="0">
+<segment>
+<pinref part="MCU_RIGHT" gate="A" pin="11"/>
+<wire x1="182.88" y1="119.38" x2="195.58" y2="119.38" width="0.1524" layer="91"/>
+<label x="185.42" y="119.38" size="1.778" layer="95"/>
+</segment>
+<segment>
+<pinref part="D_LEFT" gate="A" pin="3"/>
+<wire x1="246.38" y1="124.46" x2="233.68" y2="124.46" width="0.1524" layer="91"/>
+<label x="233.68" y="124.46" size="1.778" layer="95"/>
+</segment>
+</net>
+<net name="GND" class="0">
+<segment>
+<pinref part="MCU_RIGHT" gate="A" pin="2"/>
+<wire x1="182.88" y1="142.24" x2="190.5" y2="142.24" width="0.1524" layer="91"/>
+<pinref part="SUPPLY1" gate="GND" pin="GND"/>
+</segment>
+<segment>
+<pinref part="U_LEFT" gate="G$1" pin="2"/>
+<wire x1="246.38" y1="134.62" x2="228.6" y2="134.62" width="0.1524" layer="91"/>
+<pinref part="SUPPLY2" gate="GND" pin="GND"/>
+<wire x1="228.6" y1="134.62" x2="228.6" y2="129.54" width="0.1524" layer="91"/>
+<wire x1="228.6" y1="129.54" x2="228.6" y2="116.84" width="0.1524" layer="91"/>
+<wire x1="228.6" y1="116.84" x2="228.6" y2="114.3" width="0.1524" layer="91"/>
+<wire x1="228.6" y1="134.62" x2="228.6" y2="137.16" width="0.1524" layer="91"/>
+<junction x="228.6" y="134.62"/>
+<pinref part="U_LEFT" gate="G$1" pin="1"/>
+<wire x1="228.6" y1="137.16" x2="246.38" y2="137.16" width="0.1524" layer="91"/>
+<pinref part="D_LEFT" gate="A" pin="1"/>
+<wire x1="246.38" y1="129.54" x2="228.6" y2="129.54" width="0.1524" layer="91"/>
+<junction x="228.6" y="129.54"/>
+<pinref part="U_RIGHT" gate="G$1" pin="2"/>
+<wire x1="254" y1="134.62" x2="269.24" y2="134.62" width="0.1524" layer="91"/>
+<wire x1="269.24" y1="134.62" x2="269.24" y2="116.84" width="0.1524" layer="91"/>
+<wire x1="269.24" y1="116.84" x2="228.6" y2="116.84" width="0.1524" layer="91"/>
+<junction x="228.6" y="116.84"/>
+<pinref part="U_RIGHT" gate="G$1" pin="1"/>
+<wire x1="254" y1="137.16" x2="269.24" y2="137.16" width="0.1524" layer="91"/>
+<wire x1="269.24" y1="137.16" x2="269.24" y2="134.62" width="0.1524" layer="91"/>
+<junction x="269.24" y="134.62"/>
+</segment>
+</net>
+<net name="5V" class="0">
+<segment>
+<pinref part="MCU_RIGHT" gate="A" pin="4"/>
+<wire x1="182.88" y1="137.16" x2="198.12" y2="137.16" width="0.1524" layer="91"/>
+<pinref part="P+1" gate="VCC" pin="VCC"/>
+<wire x1="198.12" y1="137.16" x2="198.12" y2="139.7" width="0.1524" layer="91"/>
+<label x="196.596" y="142.24" size="1.778" layer="95"/>
+</segment>
+<segment>
+<pinref part="D_LEFT" gate="A" pin="4"/>
+<wire x1="246.38" y1="121.92" x2="231.14" y2="121.92" width="0.1524" layer="91"/>
+<pinref part="P+2" gate="VCC" pin="VCC"/>
+<label x="229.362" y="124.46" size="1.778" layer="95"/>
+</segment>
+</net>
 </nets>
 </sheet>
@@
 will not be understood (or retained) with this version.
 </note>
+<note version="8.3" severity="warning">
+Since Version 8.3, EAGLE supports the association of 3D packages
+with devices in libraries, schematics, and board files. Those 3D
+packages will not be understood (or retained) with this version.
+</note>
 </compatibility>
